Commit message: update joint axis orientation

File: hardware/URDF/Poppy_Humanoid/robots/Poppy_Humanoid.URDF (robot description, URDF)
Before this commit: robot Poppy_Humanoid, 26 links, 25 joints
Joints:
- joint abs_x: axis 0 0 -1 -> 0 0 1
- joint abs_y: axis 1 0 0 -> -1 0 0
- joint bust_x: axis 0 0 -1 -> 0 0 1
- joint bust_y: axis 1 0 0 -> -1 0 0
- joint head_y: axis 1 0 0 -> -1 0 0
- joint l_arm_z: axis 0 -1 0 -> 0 1 0
- joint l_hip_z: axis 0 1 0 -> 0 -1 0
- joint l_shoulder_x: axis 0 0 -1 -> 0 0 1
- joint r_ankle_y: axis 1 0 0 -> -1 0 0
- joint r_arm_z: axis 0 -1 0 -> 0 1 0
- joint r_elbow_y: axis 1 0 0 -> -1 0 0
- joint r_hip_y: axis 1 0 0 -> -1 0 0
- joint r_hip_z: axis 0 1 0 -> 0 -1 0
- joint r_knee_y: axis 0 0 -1 -> 0 0 1
- joint r_shoulder_y: axis 1 0 0 -> -1 0 0
