Commit message: update urdf path to 3D models

File: hardware/URDF/robots/Poppy_Humanoid.URDF (robot description, URDF)
Before this commit: robot Poppy_Humanoid, 26 links, 25 joints
Links:
- link abdomen: geometry collision mesh filename=package://meshes/abdomen.STL; visual mesh filename=package://meshes/abdomen.STL
- link abs_motors: geometry collision mesh filename=package://meshes/abs_motors.STL; visual mesh filename=package://meshes/abs_motors.STL
- link bust_motors: geometry collision mesh filename=package://meshes/bust_motors.STL; visual mesh filename=package://meshes/bust_motors.STL
- link chest: geometry collision mesh filename=package://meshes/chest.STL; visual mesh filename=package://meshes/chest.STL
- link head: geometry collision mesh filename=package://meshes/head.STL; visual mesh filename=package://meshes/head.STL
- link l_foot: geometry collision mesh filename=package://meshes/l_foot.STL; visual mesh filename=package://meshes/l_foot.STL
- link l_forearm: geometry collision mesh filename=package://meshes/l_forearm.STL; visual mesh filename=package://meshes/l_forearm.STL
- link l_hip: geometry collision mesh filename=package://meshes/l_hip.STL; visual mesh filename=package://meshes/l_hip.STL
- link l_hip_motor: geometry collision mesh filename=package://meshes/l_hip_motor.STL; visual mesh filename=package://meshes/l_hip_motor.STL
- link l_leg: geometry collision mesh filename=package://meshes/l_leg.STL; visual mesh filename=package://meshes/l_leg.STL
- link l_shoulder: geometry collision mesh filename=package://meshes/l_shoulder.STL; visual mesh filename=package://meshes/l_shoulder.STL
- link l_shoulder_motor: geometry collision mesh filename=package://meshes/l_shoulder_motor.STL; visual mesh filename=package://meshes/l_shoulder_motor.STL
- link l_thigh: geometry collision mesh filename=package://meshes/l_thigh.STL; visual mesh filename=package://meshes/l_thigh.STL
- link neck: geometry collision mesh filename=package://meshes/neck.STL; visual mesh filename=package://meshes/neck.STL
- link pelvis: geometry collision mesh filename=package://meshes/pelvis.STL; visual mesh filename=package://meshes/pelvis.STL
- link r_foot: geometry collision mesh filename=package://meshes/r_foot.STL; visual mesh filename=package://meshes/r_foot.STL
- link r_forearm: geometry collision mesh filename=package://meshes/r_forearm.STL; visual mesh filename=package://meshes/r_forearm.STL
- link r_hip: geometry collision mesh filename=package://meshes/r_hip.STL; visual mesh filename=package://meshes/r_hip.STL
- link r_hip_motor: geometry collision mesh filename=package://meshes/r_hip_motor.STL; visual mesh filename=package://meshes/r_hip_motor.STL
- link r_leg: geometry collision mesh filename=package://meshes/r_leg.STL; visual mesh filename=package://meshes/r_leg.STL
- link r_shoulder: geometry collision mesh filename=package://meshes/r_shoulder.STL; visual mesh filename=package://meshes/r_shoulder.STL
- link r_shoulder_motor: geometry collision mesh filename=package://meshes/r_shoulder_motor.STL; visual mesh filename=package://meshes/r_shoulder_motor.STL
- link r_thigh: geometry collision mesh filename=package://meshes/r_thigh.STL; visual mesh filename=package://meshes/r_thigh.STL
- link r_upper_arm: geometry collision mesh filename=package://meshes/r_upper_arm.STL; visual mesh filename=package://meshes/r_upper_arm.STL
- link spine: geometry collision mesh filename=package://meshes/spine.STL; visual mesh filename=package://meshes/spine.STL
- link upper_arm: geometry collision mesh filename=package://meshes/upper_arm.STL; visual mesh filename=package://meshes/upper_arm.STL

Commit message: URDF file updated

File: hardware/URDF/robots/Poppy_Humanoid.URDF (robot description, URDF)
Before this commit: robot Poppy_Humanoid, 26 links, 25 joints
Joints:
- joint abs_x: limit lower=-3 upper=3 effort=6.4 velocity=10 -> lower=-0.785398163397 upper=0.785398163397 effort=7.3 velocity=8.2
- joint abs_y: limit lower=-3 upper=3 effort=6.4 velocity=10 -> lower=-0.645771823238 upper=0.279252680319 effort=7.3 velocity=8.2
- joint abs_z: limit lower=-3 upper=3 effort=6.4 velocity=10 -> lower=-1.3962634016 upper=1.3962634016 effort=3.1 velocity=7.0
- joint bust_x: limit lower=-3 upper=3 effort=6.4 velocity=10 -> lower=-0.698131700798 upper=0.698131700798 effort=3.1 velocity=7.0
- joint bust_y: limit lower=-3 upper=3 effort=6.4 velocity=10 -> lower=-0.802851455917 upper=0.401425727959 effort=3.1 velocity=7.0
- joint head_y: limit lower=-3 upper=3 effort=6.4 velocity=10 -> lower=-0.698131700798 upper=0.13962634016 effort=1.8 velocity=10.0
- joint head_z: limit lower=-3 upper=3 effort=6.4 velocity=10 -> lower=-1.74532925199 upper=1.74532925199 effort=1.8 velocity=10.0
- joint l_ankle_y: limit lower=-3 upper=3 effort=6.4 velocity=10 -> lower=-0.610865238198 upper=1.2217304764 effort=3.1 velocity=7.0
- joint l_arm_z: limit lower=-3 upper=3 effort=6.4 velocity=10 -> lower=-1.57079632679 upper=1.57079632679 effort=3.1 velocity=7.0
- joint l_elbow_y: limit lower=-3 upper=3 effort=6.4 velocity=10 -> lower=-2.44346095279 upper=0.0 effort=3.1 velocity=7.0
- joint l_hip_x: limit lower=-3 upper=3 effort=6.4 velocity=10 -> lower=-0.383972435439 upper=0.785398163397 effort=3.1 velocity=7.0
- joint l_hip_y: limit lower=-3 upper=3 effort=6.4 velocity=10 -> lower=-1.83259571459 upper=1.4835298642 effort=7.3 velocity=8.2
- joint l_hip_z: limit lower=-3 upper=3 effort=6.4 velocity=10 -> lower=-0.698131700798 upper=0.436332312999 effort=3.1 velocity=7.0
- joint l_knee_y: limit lower=-3 upper=3 effort=6.4 velocity=10 -> lower=-0.0349065850399 upper=2.09439510239 effort=3.1 velocity=7.0
- joint l_shoulder_x: limit lower=-3 upper=3 effort=6.4 velocity=10 -> lower=-1.83259571459 upper=1.91986217719 effort=3.1 velocity=7.0
- joint l_shoulder_y: limit lower=-3 upper=3 effort=6.4 velocity=10 -> lower=-2.09439510239 upper=2.70526034059 effort=3.1 velocity=7.0
- joint r_ankle_y: limit lower=-3 upper=3 effort=6.4 velocity=10 -> lower=-1.2217304764 upper=0.436332312999 effort=3.1 velocity=7.0
- joint r_arm_z: limit lower=-3 upper=3 effort=6.4 velocity=10 -> lower=-1.57079632679 upper=1.57079632679 effort=3.1 velocity=7.0
- joint r_elbow_y: limit lower=-3 upper=3 effort=6.4 velocity=10 -> lower=0.0 upper=2.56563400043 effort=3.1 velocity=7.0
- joint r_hip_x: limit lower=-3 upper=3 effort=6.4 velocity=10 -> lower=-0.785398163397 upper=0.349065850399 effort=3.1 velocity=7.0
- joint r_hip_y: limit lower=-3 upper=3 effort=6.4 velocity=10 -> lower=-1.4835298642 upper=1.83259571459 effort=7.3 velocity=8.2
- joint r_hip_z: limit lower=-3 upper=3 effort=6.4 velocity=10 -> lower=-0.436332312999 upper=0.698131700798 effort=3.1 velocity=7.0
- joint r_knee_y: axis 0 0 1 -> 0 0 -1; limit lower=-3 upper=3 effort=6.4 velocity=10 -> lower=-2.09439510239 upper=0.0349065850399 effort=3.1 velocity=7.0
- joint r_shoulder_x: limit lower=-3 upper=3 effort=6.4 velocity=10 -> lower=-1.91986217719 upper=1.83259571459 effort=3.1 velocity=7.0
- joint r_shoulder_y: limit lower=-3 upper=3 effort=6.4 velocity=10 -> lower=-2.70526034059 upper=2.09439510239 effort=3.1 velocity=7.0

Commit message: rebuild of every shapes and modify URDF file

File: hardware/URDF/robots/Poppy_Humanoid.URDF (robot description, URDF)
Before this commit: robot Poppy_Humanoid, 26 links, 25 joints
Links:
- removed link l_leg
- removed link r_leg
- removed link upper_arm
- added link l_shin, mass 0.11558221959692; collision mesh filename=package://meshes/l_shin_respondable.STL; visual mesh filename=package://meshes/l_shin.STL
- added link l_upper_arm, mass 0.168140859572398; collision mesh filename=package://meshes/l_upper_arm_respondable.STL; visual mesh filename=package://meshes/l_upper_arm.STL
- added link r_shin, mass 0.115582219792398; collision mesh filename=package://meshes/r_shin_respondable.STL; visual mesh filename=package://meshes/r_shin.STL
- link abdomen: geometry collision mesh filename=package://meshes/abdomen_respondable.STL; visual mesh filename=package://meshes/abdomen.STL
- link abs_motors: geometry collision mesh filename=package://meshes/abs_motors_respondable.STL; visual mesh filename=package://meshes/abs_motors.STL
- link bust_motors: geometry collision mesh filename=package://meshes/bust_motors_respondable.STL; visual mesh filename=package://meshes/bust_motors.STL
- link chest: geometry collision mesh filename=package://meshes/chest_respondable.STL; visual mesh filename=package://meshes/chest.STL
- link head: geometry collision mesh filename=package://meshes/head_respondable.STL; visual mesh filename=package://meshes/head.STL
- link l_foot: geometry collision mesh filename=package://meshes/l_foot_respondable.STL; visual mesh filename=package://meshes/l_foot.STL
- link l_forearm: geometry collision mesh filename=package://meshes/l_forearm_respondable.STL; visual mesh filename=package://meshes/l_forearm.STL
- link l_hip: geometry collision mesh filename=package://meshes/l_hip_respondable.STL; visual mesh filename=package://meshes/l_hip.STL
- link l_hip_motor: geometry collision mesh filename=package://meshes/l_hip_motor_respondable.STL; visual mesh filename=package://meshes/l_hip_motor.STL
- link l_shoulder: geometry collision mesh filename=package://meshes/l_shoulder_respondable.STL; visual mesh filename=package://meshes/l_shoulder.STL
- link l_shoulder_motor: geometry collision mesh filename=package://meshes/l_shoulder_motor_respondable.STL; visual mesh filename=package://meshes/l_shoulder_motor.STL
- link l_thigh: geometry collision mesh filename=package://meshes/l_thigh_respondable.STL; visual mesh filename=package://meshes/l_thigh.STL
- link neck: geometry collision mesh filename=package://meshes/neck_respondable.STL; visual mesh filename=package://meshes/neck.STL
- link pelvis: geometry collision mesh filename=package://meshes/pelvis_respondable.STL; visual mesh filename=package://meshes/pelvis.STL
- link r_foot: geometry collision mesh filename=package://meshes/r_foot_respondable.STL; visual mesh filename=package://meshes/r_foot.STL
- link r_forearm: geometry collision mesh filename=package://meshes/r_forearm_respondable.STL; visual mesh filename=package://meshes/r_forearm.STL
- link r_hip: geometry collision mesh filename=package://meshes/r_hip_respondable.STL; visual mesh filename=package://meshes/r_hip.STL
- link r_hip_motor: geometry collision mesh filename=package://meshes/r_hip_motor_respondable.STL; visual mesh filename=package://meshes/r_hip_motor.STL
- link r_shoulder: geometry collision mesh filename=package://meshes/r_shoulder_respondable.STL; visual mesh filename=package://meshes/r_shoulder.STL
- link r_shoulder_motor: geometry collision mesh filename=package://meshes/r_shoulder_motor_respondable.STL; visual mesh filename=package://meshes/r_shoulder_motor.STL
- link r_thigh: geometry collision mesh filename=package://meshes/r_thigh_respondable.STL; visual mesh filename=package://meshes/r_thigh.STL
- link r_upper_arm: geometry collision mesh filename=package://meshes/r_upper_arm_respondable.STL; visual mesh filename=package://meshes/r_upper_arm.STL
- link spine: geometry collision mesh filename=package://meshes/spine_respondable.STL; visual mesh filename=package://meshes/spine.STL
Joints:
- joint l_ankle_y: parent l_leg -> l_shin
- joint l_arm_z: child upper_arm -> l_upper_arm
- joint l_elbow_y: parent upper_arm -> l_upper_arm
- joint l_knee_y: child l_leg -> l_shin
- joint r_ankle_y: parent r_leg -> r_shin
- joint r_knee_y: child r_leg -> r_shin

Commit message: update URDF robot angle limits

File: hardware/URDF/robots/Poppy_Humanoid.URDF (robot description, URDF)
Before this commit: robot Poppy_Humanoid, 26 links, 25 joints
Joints:
- joint abs_y: limit lower=-0.645771823238 upper=0.279252680319 effort=7.3 velocity=8.2 -> lower=-0.872664625997 upper=0.209439510239 effort=7.3 velocity=8.2
- joint abs_z: limit lower=-1.3962634016 upper=1.3962634016 effort=3.1 velocity=7.0 -> lower=-1.57079632679 upper=1.57079632679 effort=3.1 velocity=7.0
- joint bust_y: limit lower=-0.802851455917 upper=0.401425727959 effort=3.1 velocity=7.0 -> lower=-1.16937059884 upper=0.471238898038 effort=3.1 velocity=7.0
- joint head_y: limit lower=-0.698131700798 upper=0.13962634016 effort=1.8 velocity=10.0 -> lower=-0.785398163397 upper=0.10471975512 effort=1.8 velocity=10.0
- joint head_z: limit lower=-1.74532925199 upper=1.74532925199 effort=1.8 velocity=10.0 -> lower=-1.57079632679 upper=1.57079632679 effort=1.8 velocity=10.0
- joint l_ankle_y: limit lower=-0.610865238198 upper=1.2217304764 effort=3.1 velocity=7.0 -> lower=-0.785398163397 upper=0.785398163397 effort=3.1 velocity=7.0
- joint l_arm_z: limit lower=-1.57079632679 upper=1.57079632679 effort=3.1 velocity=7.0 -> lower=-1.83259571459 upper=1.83259571459 effort=3.1 velocity=7.0
- joint l_elbow_y: limit lower=-2.44346095279 upper=0.0 effort=3.1 velocity=7.0 -> lower=-2.58308729295 upper=0.0174532925199 effort=3.1 velocity=7.0
- joint l_hip_x: limit lower=-0.383972435439 upper=0.785398163397 effort=3.1 velocity=7.0 -> lower=-0.523598775598 upper=0.497418836818 effort=3.1 velocity=7.0
- joint l_hip_y: limit lower=-1.83259571459 upper=1.4835298642 effort=7.3 velocity=8.2 -> lower=-1.81514242207 upper=1.46607657168 effort=7.3 velocity=8.2
- joint l_hip_z: limit lower=-0.698131700798 upper=0.436332312999 effort=3.1 velocity=7.0 -> lower=-0.436332312999 upper=1.57079632679 effort=3.1 velocity=7.0
- joint l_knee_y: limit lower=-0.0349065850399 upper=2.09439510239 effort=3.1 velocity=7.0 -> lower=-0.0610865238198 upper=2.33874119767 effort=3.1 velocity=7.0
- joint r_ankle_y: limit lower=-1.2217304764 upper=0.436332312999 effort=3.1 velocity=7.0 -> lower=-0.785398163397 upper=0.785398163397 effort=3.1 velocity=7.0
- joint r_arm_z: limit lower=-1.57079632679 upper=1.57079632679 effort=3.1 velocity=7.0 -> lower=-1.83259571459 upper=1.83259571459 effort=3.1 velocity=7.0
- joint r_elbow_y: limit lower=0.0 upper=2.56563400043 effort=3.1 velocity=7.0 -> lower=-0.0174532925199 upper=2.58308729295 effort=3.1 velocity=7.0
- joint r_hip_x: limit lower=-0.785398163397 upper=0.349065850399 effort=3.1 velocity=7.0 -> lower=-0.497418836818 upper=0.523598775598 effort=3.1 velocity=7.0
- joint r_hip_z: limit lower=-0.436332312999 upper=0.698131700798 effort=3.1 velocity=7.0 -> lower=-1.57079632679 upper=0.436332312999 effort=3.1 velocity=7.0
- joint r_knee_y: limit lower=-2.09439510239 upper=0.0349065850399 effort=3.1 velocity=7.0 -> lower=-2.33874119767 upper=0.0610865238198 effort=3.1 velocity=7.0
